Commit message: feat: finalizando robo

File: urdf/rosbot3.xacro (robot description, xacro)
@@ -5,40 +5,100 @@
 -->
 <robot name="rosbot3" xmlns:xacro="http://www.ros.org/wiki/xacro">
-  <xacro:include filename="$(find rosbot3_description)/urdf/ugv02.xacro"/>
-  <xacro:property name="payload_base_length" value="${130 * M}"/>
-  <xacro:property name="payload_base_width" value="${130 * M}"/>
-  <xacro:property name="payload_base_height" value="${38 * M}"/>
-  <xacro:property name="lidar_side" value="${45.61 * M}"/>
-  <xacro:property name="lidar_height" value="${38 * M}"/>
+  <xacro:include filename="$(find rosbot3_description)/urdf/ugv02.xacro" />
+  <xacro:property name="payload_base_length" value="${130 * M}" />
+  <xacro:property name="payload_base_width" value="${130 * M}" />
+  <xacro:property name="payload_base_height" value="${38 * M}" />
+  <xacro:property name="camera_vertical_base_length" value="${20 * M}" />
+  <xacro:property name="camera_vertical_base_width" value="${3 * M}" />
+  <xacro:property name="camera_vertical_base_height" value="${94 * M}" />
+  <xacro:property name="camera_horizontal_base_length" value="${35 * M}" />
+  <xacro:property name="camera_horizontal_base_width" value="${3 * M}" />
+  <xacro:property name="camera_horizontal_base_height" value="${20 * M}" />
+  <xacro:property name="camera_length" value="${20 * M}" />
+  <xacro:property name="camera_width" value="${80 * M}" />
+  <xacro:property name="camera_height" value="${30 * M}" />
+  <xacro:property name="lidar_radius" value="${50 * M}" />
+  <xacro:property name="lidar_height" value="${38 * M}" />
+  <xacro:property name="antenna_radius" value="${5 * M}" />
+  <xacro:property name="antenna_height" value="${80 * M}" />
   <xacro:solid_block
-    name="payload_base"
-    size_x="${payload_base_length}"
-    size_y="${payload_base_width}"
-    size_z="${payload_base_height}"
+    name="camera_vertical_right_base"
+    size_x="${camera_vertical_base_length}"
+    size_y="${camera_vertical_base_width}"
+    size_z="${camera_vertical_base_height}"
+  />
+  <xacro:solid_block
+    name="camera_vertical_left_base"
+    size_x="${camera_vertical_base_length}"
+    size_y="${camera_vertical_base_width}"
+    size_z="${camera_vertical_base_height}"
   />
   <xacro:joint_fixed
     parent="body"
-    child="payload_base"
-    z="${0.5 * (body_height + payload_base_height)}"
+    child="camera_vertical_left_base"
+    x="${-0.3 * body_length}"
+    y="${0.2 * body_width}"
+    z="${0.5 * (body_height + camera_vertical_base_height)}"
   />
-  <xacro:camera_link name="camera_front"/>
   <xacro:joint_fixed
-    parent="payload_base"
-    child="camera_front"
-    x="${0.5 * payload_base_length}"
+    parent="body"
+    child="camera_vertical_right_base"
+    x="${-0.3 * body_length}"
+    y="${-0.2 * body_width}"
+    z="${0.5 * (body_height + camera_vertical_base_height)}"
   />
   <xacro:solid_block
-    name="lidar"
-    size_x="${lidar_side}"
-    size_y="${lidar_side}"
-    size_z="${lidar_height}"
+    name="camera_horizontal_left_base"
+    size_x="${camera_horizontal_base_length}"
+    size_y="${camera_horizontal_base_width}"
+    size_z="${camera_horizontal_base_height}"
+  />
+  <xacro:solid_block
+    name="camera_horizontal_right_base"
+    size_x="${camera_horizontal_base_length}"
+    size_y="${camera_horizontal_base_width}"
+    size_z="${camera_horizontal_base_height}"
   />
   <xacro:joint_fixed
-    parent="payload_base"
+    parent="camera_vertical_left_base"
+    child="camera_horizontal_left_base"
+    x="${camera_vertical_base_length}"
+    z="${0.5 * (camera_vertical_base_height - camera_horizontal_base_height)}"
+  />
+  <xacro:joint_fixed
+    parent="camera_vertical_right_base"
+    child="camera_horizontal_right_base"
+    x="${camera_vertical_base_length}"
+    z="${0.5 * (camera_vertical_base_height - camera_horizontal_base_height)}"
+  />
+  <xacro:solid_block
+    name="camera"
+    size_x="${camera_length}"
+    size_y="${camera_width}"
+    size_z="${camera_height}"
+  />
+  <xacro:joint_fixed
+    parent="camera_horizontal_right_base"
+    child="camera"
+    x="${0.5 * camera_length}"
+    y="${0.5*camera_width - 3.4 * M}"
+  />
+  <xacro:camera_link name="camera_front" />
+  <xacro:joint_fixed
+    parent="camera"
+    child="camera_front"
+    x="${0.5 * camera_length}"
+  />
+  <xacro:solid_cylinder
+    name="lidar"
+    length="${lidar_height}"
+    radius="${lidar_radius}"
+  />
+  <xacro:joint_fixed
+    parent="body"
     child="lidar"
-    x="${0.5 * payload_base_height}"
-    z="${0.5 * (payload_base_height + lidar_height)}"
+    z="${0.5 * (body_height + lidar_height)}"
   />
-  <link name="laser"/>
+  <link name="laser" />
   <xacro:joint_fixed
     parent="lidar"
@@ -46,3 +106,15 @@
     z="${0.5 * lidar_height}"
   />
+    <xacro:solid_cylinder
+    name="antenna"
+    length="${antenna_height}"
+    radius="${antenna_radius}"
+  />
+  <xacro:joint_fixed
+    parent="body"
+    child="antenna"
+    x="${-0.45 * body_length}"
+    y="${0.2 * body_width}"
+    z="${0.5 * (body_height + antenna_height)}"
+  />
 </robot>

File: urdf/ugv02.xacro (robot description, xacro)
@@ -27,5 +27,5 @@
   <xacro:property name="fender_side_width" value="${wheel_radius + fender_thickness + fender_top_gap}"/>
   <xacro:property name="fender_side_y_offset" value="${0.5 * (fender_top_width + fender_thickness)}"/>
-  <xacro:property name="fender_side_z_offset" value="${0.5 * (fender_thickness - fender_side_width)}"/> --> -->
+  <xacro:property name="fender_side_z_offset" value="${0.5 * (fender_thickness - fender_side_width)}"/> -->
   <xacro:property name="wheel_axle_z_offset" value="${wheel_radius - 0.5 * body_height - ground_clearance}"/>
   <xacro:macro

Commit message: feat: commenting antenna and adding info comments to the code

File: urdf/rosbot3.xacro (robot description, xacro)
@@ -6,7 +6,5 @@
 <robot name="rosbot3" xmlns:xacro="http://www.ros.org/wiki/xacro">
   <xacro:include filename="$(find rosbot3_description)/urdf/ugv02.xacro" />
-  <xacro:property name="payload_base_length" value="${130 * M}" />
-  <xacro:property name="payload_base_width" value="${130 * M}" />
-  <xacro:property name="payload_base_height" value="${38 * M}" />
+  <!-- Dimensions of the camera base -->
   <xacro:property name="camera_vertical_base_length" value="${20 * M}" />
   <xacro:property name="camera_vertical_base_width" value="${3 * M}" />
@@ -15,11 +13,15 @@
   <xacro:property name="camera_horizontal_base_width" value="${3 * M}" />
   <xacro:property name="camera_horizontal_base_height" value="${20 * M}" />
+  <!-- Dimensions of the camera -->
   <xacro:property name="camera_length" value="${20 * M}" />
   <xacro:property name="camera_width" value="${80 * M}" />
   <xacro:property name="camera_height" value="${30 * M}" />
+<!-- Dimensions of the lidar -->
   <xacro:property name="lidar_radius" value="${50 * M}" />
   <xacro:property name="lidar_height" value="${38 * M}" />
-  <xacro:property name="antenna_radius" value="${5 * M}" />
-  <xacro:property name="antenna_height" value="${80 * M}" />
+  <!-- Dimensions of the antenna-->
+  <!-- <xacro:property name="antenna_radius" value="${5 * M}" />
+  <xacro:property name="antenna_height" value="${80 * M}" /> -->
+  <!-- Building the vertical part of the camera base for both sides-->
   <xacro:solid_block
     name="camera_vertical_right_base"
@@ -34,4 +36,5 @@
     size_z="${camera_vertical_base_height}"
   />
+  <!-- Joining the vertical camera base to the body of the robot for both sides-->
   <xacro:joint_fixed
     parent="body"
@@ -48,4 +51,5 @@
     z="${0.5 * (body_height + camera_vertical_base_height)}"
   />
+  <!-- Building the horizontal part of the camera base for both sides-->
   <xacro:solid_block
     name="camera_horizontal_left_base"
@@ -60,4 +64,5 @@
     size_z="${camera_horizontal_base_height}"
   />
+  <!-- Joining the horizontal camera base to the vertical camera base for both sides-->
   <xacro:joint_fixed
     parent="camera_vertical_left_base"
@@ -72,4 +77,5 @@
     z="${0.5 * (camera_vertical_base_height - camera_horizontal_base_height)}"
   />
+  <!-- Building the camera structure -->
   <xacro:solid_block
     name="camera"
@@ -78,4 +84,5 @@
     size_z="${camera_height}"
   />
+  <!-- Joining the camera to the horizontal camera base-->
   <xacro:joint_fixed
     parent="camera_horizontal_right_base"
@@ -84,5 +91,7 @@
     y="${0.5*camera_width - 3.4 * M}"
   />
+  <!-- Creating the camera link -->
   <xacro:camera_link name="camera_front" />
+  <!-- Joining the camera link to the camera's structure (block) -->
   <xacro:joint_fixed
     parent="camera"
@@ -90,4 +99,5 @@
     x="${0.5 * camera_length}"
   />
+  <!-- Building the lidar structure -->
   <xacro:solid_cylinder
     name="lidar"
@@ -95,4 +105,5 @@
     radius="${lidar_radius}"
   />
+  <!-- Joining the lidar to the body of the robot-->
   <xacro:joint_fixed
     parent="body"
@@ -100,5 +111,7 @@
     z="${0.5 * (body_height + lidar_height)}"
   />
+  <!-- Creating the lidar/laser link -->
   <link name="laser" />
+  <!-- Joining the lidar/laser link to the lidar's structure (cylinder) --> -->
   <xacro:joint_fixed
     parent="lidar"
@@ -106,10 +119,12 @@
     z="${0.5 * lidar_height}"
   />
-    <xacro:solid_cylinder
+  <!-- Building the antenna structure -->
+    <!-- <xacro:solid_cylinder
     name="antenna"
     length="${antenna_height}"
     radius="${antenna_radius}"
-  />
-  <xacro:joint_fixed
+  /> -->
+  <!-- Joining the antenna to the body of the robot-->
+  <!-- <xacro:joint_fixed
     parent="body"
     child="antenna"
@@ -117,4 +132,6 @@
     y="${0.2 * body_width}"
     z="${0.5 * (body_height + antenna_height)}"
-  />
+  /> -->
 </robot>
+<!-- PS: I commented the antenna because the lidar is geting its position in the rviz, so I don't know if it's worth to let it there.
+ Maybe it is a calibration issue. If you want to see with it, just uncomment the dimensions, the building of the solid_cylinder and the joints -->

File: urdf/ugv02.xacro (robot description, xacro)
@@ -5,28 +5,22 @@
 -->
 <robot xmlns:xacro="http://www.ros.org/wiki/xacro">
-  <xacro:include filename="$(find ros_commons)/urdf/domain.xacro"/>
-  <xacro:property name="M" value="0.001"/>
-  <xacro:property name="overall_height" value="${103 * M}"/>
+  <xacro:include filename="$(find ros_commons)/urdf/domain.xacro" />
+  <xacro:property name="M" value="0.001" />
+  <xacro:property name="overall_height" value="${103 * M}" />
   <!-- Using standard wheels values -->
-  <xacro:property name="ground_clearance" value="${23 * M}"/>
-  <xacro:property name="wheel_diameter" value="${84.0 * M}"/>
-  <xacro:property name="wheel_radius" value="${0.5 * wheel_diameter}"/>
-  <xacro:property name="wheelbase" value="${106.0 * M}"/>
+  <xacro:property name="ground_clearance" value="${23 * M}" />
+  <xacro:property name="wheel_diameter" value="${84.0 * M}" />
+  <xacro:property name="wheel_radius" value="${0.5 * wheel_diameter}" />
+  <xacro:property name="wheelbase" value="${106.0 * M}" />
   <!-- Value not defined. Random value put from image -->
-  <xacro:property name="wheel_thickness" value="${25 * M}"/>
+  <xacro:property name="wheel_thickness" value="${25 * M}" />
   <!-- Distance between intern part of both wheels in the same axe -->
-  <xacro:property name="wheel_separation" value="${233.0 * M - 2* wheel_thickness}"/>
-  <xacro:property name="body_length" value="${200.0 * M}"/>
-  <xacro:property name="body_width" value="${233.0 * M - 2 * wheel_thickness}"/>
-  <xacro:property name="body_height" value="${103.0 * M - ground_clearance }"/>
-  <!-- <xacro:property name="fender_length" value="${200.0 * M}"/>
-  <xacro:property name="fender_thickness" value="${3.0 * M}"/>
-  <xacro:property name="fender_top_gap" value="${1.0 * M}"/>
-  <xacro:property name="fender_side_gap" value="${5.0 * M}"/>
-  <xacro:property name="fender_top_width" value="${body_width + 2.0 * (wheel_thickness * 0.75)}"/>
-  <xacro:property name="fender_side_width" value="${wheel_radius + fender_thickness + fender_top_gap}"/>
-  <xacro:property name="fender_side_y_offset" value="${0.5 * (fender_top_width + fender_thickness)}"/>
-  <xacro:property name="fender_side_z_offset" value="${0.5 * (fender_thickness - fender_side_width)}"/> -->
-  <xacro:property name="wheel_axle_z_offset" value="${wheel_radius - 0.5 * body_height - ground_clearance}"/>
+  <xacro:property name="wheel_separation" value="${233.0 * M - 2* wheel_thickness}" />
+  <xacro:property name="body_length" value="${200.0 * M}" />
+  <xacro:property name="body_width" value="${233.0 * M - 2 * wheel_thickness}" />
+  <xacro:property name="body_height" value="${103.0 * M - ground_clearance }" />
+  <xacro:property name="wheel_axle_z_offset"
+    value="${wheel_radius - 0.5 * body_height - ground_clearance}" />
+  <!-- Using roselito's macro to generate the axles and wheels-->
   <xacro:macro
     name="wheels"
@@ -66,6 +60,8 @@
     />
   </xacro:macro>
-  <xacro:wheels position="front"/>
-  <xacro:wheels position="rear"/>
+  <!-- Generating wheels and axles-->
+  <xacro:wheels position="front" />
+  <xacro:wheels position="rear" />
+  <!-- Building the body structure-->
   <xacro:solid_block
     name="body"
@@ -74,4 +70,5 @@
     size_z="${body_height}"
   />
+  <!-- Joining the axles to the body-->
   <xacro:joint_fixed
     parent="body"
@@ -86,5 +83,7 @@
     z="${wheel_axle_z_offset}"
   />
-  <link name="base_link"/>
+  <!-- Creating the base link-->
+  <link name="base_link" />
+  <!-- Joining the base link to the body-->
   <xacro:joint_fixed
     parent="base_link"

Commit message: feat: adicionando medidas certas do lidar e da camera

File: urdf/rosbot3.xacro (robot description, xacro)
@@ -9,15 +9,20 @@
   <xacro:property name="camera_vertical_base_length" value="${20 * M}" />
   <xacro:property name="camera_vertical_base_width" value="${3 * M}" />
-  <xacro:property name="camera_vertical_base_height" value="${94 * M}" />
+  <xacro:property name="camera_vertical_base_height" value="${70 * M}" />
   <xacro:property name="camera_horizontal_base_length" value="${35 * M}" />
   <xacro:property name="camera_horizontal_base_width" value="${3 * M}" />
   <xacro:property name="camera_horizontal_base_height" value="${20 * M}" />
-  <!-- Dimensions of the camera -->
-  <xacro:property name="camera_length" value="${20 * M}" />
-  <xacro:property name="camera_width" value="${80 * M}" />
-  <xacro:property name="camera_height" value="${30 * M}" />
-<!-- Dimensions of the lidar -->
-  <xacro:property name="lidar_radius" value="${50 * M}" />
-  <xacro:property name="lidar_height" value="${38 * M}" />
+  <!-- Dimensions of the camera OAK-D Lite-->
+   <!-- https://shop.luxonis.com/products/oak-d-lite-1?variant=42583102456031 -->
+  <xacro:property name="camera_length" value="${17.5 * M}" />
+  <xacro:property name="camera_width" value="${91 * M}" />
+  <xacro:property name="camera_height" value="${28 * M}" />
+  <!-- Dimensions of the lidar RPLIDAR C1
+   contained in this link
+   https://bucket-download.slamtec.com/2d4664be9f9f5c748f3b608f2cf1862962b168eb/SLAMTEC_rplidar_datasheet_C1_v1.1_en.pdf-->
+  <xacro:property name="lidar_base_side" value="${55.6 * M}" />
+  <xacro:property name="lidar_base_height" value="${23.1 * M}" />
+  <xacro:property name="lidar_radius" value="${27 * M}" />
+  <xacro:property name="lidar_height" value="${18.2 * M}" />
   <!-- Dimensions of the antenna-->
   <!-- <xacro:property name="antenna_radius" value="${5 * M}" />
@@ -40,5 +45,4 @@
     parent="body"
     child="camera_vertical_left_base"
-    x="${-0.3 * body_length}"
     y="${0.2 * body_width}"
     z="${0.5 * (body_height + camera_vertical_base_height)}"
@@ -47,5 +51,4 @@
     parent="body"
     child="camera_vertical_right_base"
-    x="${-0.3 * body_length}"
     y="${-0.2 * body_width}"
     z="${0.5 * (body_height + camera_vertical_base_height)}"
@@ -89,5 +92,5 @@
     child="camera"
     x="${0.5 * camera_length}"
-    y="${0.5*camera_width - 3.4 * M}"
+    y="${0.5*camera_width - 8.9 * M}"
   />
   <!-- Creating the camera link -->
@@ -99,4 +102,21 @@
     x="${0.5 * camera_length}"
   />
+  <!-- Building the lidar base structure -->
+  <xacro:solid_block
+    name="lidar_base"
+    size_x="${lidar_base_side}"
+    size_y="${lidar_base_side}"
+    size_z="${lidar_base_height}"
+  />
+  <!-- Joining the lidar to the body of the robot-->
+  <xacro:joint_fixed
+    parent="body"
+    child="lidar_base"
+    z="${0.5 * (body_height + lidar_base_height)- 3.3*M}"
+    x="${0.2 * body_length}"
+  />
+<!-- I subtracted 3.3 in z because at the lidar datasheet, the height is 3.3 higher than
+  in the ROSbot3 documentation. So I supposed that the lidar is a bit drownedin the robot surface.
+-->
   <!-- Building the lidar structure -->
   <xacro:solid_cylinder
@@ -107,7 +127,7 @@
   <!-- Joining the lidar to the body of the robot-->
   <xacro:joint_fixed
-    parent="body"
+    parent="lidar_base"
     child="lidar"
-    z="${0.5 * (body_height + lidar_height)}"
+    z="${0.5 * (lidar_base_height + lidar_height)}"
   />
   <!-- Creating the lidar/laser link -->

File: urdf/ugv02.xacro (robot description, xacro)
@@ -20,4 +20,9 @@
   <xacro:property name="body_width" value="${233.0 * M - 2 * wheel_thickness}" />
   <xacro:property name="body_height" value="${103.0 * M - ground_clearance }" />
+  <!-- Value not defined. Random value put from image-->
+   <!-- Fender that covers the top view of the wheels -->
+  <xacro:property name="fender_length" value="${200.0 * M}" />
+  <xacro:property name="fender_width" value="${233.0 * M }" />
+  <xacro:property name="fender_height" value="${2 * M }" />
   <xacro:property name="wheel_axle_z_offset"
     value="${wheel_radius - 0.5 * body_height - ground_clearance}" />
@@ -83,4 +88,16 @@
     z="${wheel_axle_z_offset}"
   />
+   <!-- Building the fender structure-->
+  <xacro:solid_block
+    name="fender"
+    size_x="${fender_length}"
+    size_y="${fender_width}"
+    size_z="${fender_height}"
+  />
+    <xacro:joint_fixed
+    parent="body"
+    child="fender"
+    z="${0.5 * body_height }"
+  />
   <!-- Creating the base link-->
   <link name="base_link" />
